File: Hardware/PCB design/TO52/Schematics_backup2.brd (EAGLE design)
At the start: 379.4 x 344.2 mm, 13 parts, among them X1 Boutons, X2 Potentiometres

Commit message: Avancement du rapport
Other:
- board size 379.4 x 344.2 mm -> 89.8 x 149.8 mm
Changed lines of the file:
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@@
 <board>
 <plain>
-<wire x1="-187.96" y1="-92.71" x2="191.44" y2="-147.32" width="0" layer="20"/>
-<wire x1="191.44" y1="-147.32" x2="167.31" y2="196.84" width="0" layer="20"/>
-<wire x1="167.31" y1="196.84" x2="-177.8" y2="181.6" width="0" layer="20"/>
-<wire x1="-177.8" y1="181.6" x2="-187.96" y2="-92.71" width="0" layer="20"/>
+<wire x1="-10.16" y1="-12.7" x2="79.68" y2="-12.7" width="0" layer="20"/>
+<wire x1="79.68" y1="-12.7" x2="79.68" y2="137.15" width="0" layer="20"/>
+<wire x1="79.68" y1="137.15" x2="-10.16" y2="137.15" width="0" layer="20"/>
+<wire x1="-10.16" y1="137.15" x2="-10.16" y2="-12.7" width="0" layer="20"/>
 </plain>
 <attributes>
